File: wireless-power/wireless-power.kicad_pcb (KiCad board)
At the start: 2 copper layers, 75.9 x 40 mm, 16 parts, among them J1 Screw_Terminal_01x01, J2 Screw_Terminal_01x01, U1 TPS62112RSAR, U2 NE555DR, U3 PBSS4480X

Commit message: changed coil terminal
Connections:
- C6 pad 2: /Coil_Low -> /+5V
- U3 pad 2: /Coil_Low -> /+5V
Changed lines of the file:
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@@
 	(net 9 "Net-(U2-OUT)")
 	(net 10 "Net-(U2-DISCH)")
-	(net 11 "/Coil_Low")
-	(net 12 "Net-(U3-BASE)")
+	(net 11 "Net-(U3-BASE)")
 	(footprint "wireless-power-footprints:QFN65P400X400X100-17N"
 		(layer "F.Cu")
@@
 			(size 0.5588 0.3048)
 			(layers "F.Cu" "F.Paste" "F.Mask")
-			(net 11 "/Coil_Low")
+			(net 3 "/+5V")
 			(pintype "unspecified")
 		)
@@
 			(size 0.755599 0.799998)
 			(layers "F.Cu" "F.Paste" "F.Mask")
-			(net 12 "Net-(U3-BASE)")
+			(net 11 "Net-(U3-BASE)")
 			(pintype "unspecified")
 		)
@@
 			(size 0.4826 1.6383)
 			(layers "F.Cu" "F.Paste" "F.Mask")
-			(net 11 "/Coil_Low")
+			(net 3 "/+5V")
 			(pinfunction "COLLECTOR")
 			(pintype "unspecified")
@@
 			(size 0.4826 1.6383)
 			(layers "F.Cu" "F.Paste" "F.Mask")
-			(net 12 "Net-(U3-BASE)")
+			(net 11 "Net-(U3-BASE)")
 			(pinfunction "BASE")
 			(pintype "unspecified")
@@
 		(fill solid)
 		(layer "F.Cu")
-		(net 12)
+		(net 11)
 	)
 	(gr_rect
@@
 		(fill solid)
 		(layer "F.Cu")
-		(net 11)
+		(net 3)
 	)
 	(gr_poly
@@
 		(fill solid)
 		(layer "F.Cu")
-		(net 12)
+		(net 11)
 	)
 	(gr_rect

Commit message: finalized transmitter PCB
Parts:
- added +5V: TestPoint, TestPoint:TestPoint_THTPad_1.0x1.0mm_Drill0.5mm, F.Cu at (139.8, 60.1)
- added Coil1: TestPoint, TestPoint:TestPoint_THTPad_1.0x1.0mm_Drill0.5mm, F.Cu at (147.5, 84.9)
- added Coil2: TestPoint, TestPoint:TestPoint_THTPad_1.0x1.0mm_Drill0.5mm, F.Cu at (147.5, 88.9)
- added G***: LOGO, LOGO, F.Cu at (148.8, 63.0)
- added GND: TestPoint, TestPoint:TestPoint_THTPad_1.0x1.0mm_Drill0.5mm, F.Cu at (114.7, 60.3)
- C4: value 40pF -> 39pF; footprint wireless-power-footprints:CAPC0603X33N -> wireless-power-footprints:CAPC6333_33N_KEM
Routing:
- net /+5V: track 5.26 -> 52.3 mm, vias 0 -> 2
- net GND: track 78.1 -> 82.7 mm

Commit message: finished receiver test board
Parts:
- renumbered Coil1 to TP1, Coil2 to TP2, +5V to TP3, GND to TP4
Routing:
- net Net-(U2-OUT): track 0.00 -> 9.12 mm
