File: wireless-power/wireless-power.kicad_pcb (KiCad board)
At the start: 2 copper layers, 75.9 x 40 mm, 21 parts, among them J1 Screw_Terminal_01x01, J2 Screw_Terminal_01x01, U1 TPS62112RSAR, U2 NE555DR, U3 PBSS4480X

Commit message: updated buck converter
Connections:
- C3 pad 2: Net-(U1-FB) -> GND
- U1 pad 10: Net-(U1-FB) -> /+5V
Changed lines of the file:
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@@
 	(net 2 "/+9V")
 	(net 3 "/+5V")
-	(net 4 "Net-(U1-FB)")
-	(net 5 "Net-(U2-THRES)")
-	(net 6 "Net-(U2-CONT)")
-	(net 7 "Net-(U1-SW)")
-	(net 8 "Net-(U1-PG)")
-	(net 9 "Net-(U2-OUT)")
-	(net 10 "Net-(U2-DISCH)")
-	(net 11 "Net-(U3-BASE)")
+	(net 4 "Net-(U2-THRES)")
+	(net 5 "Net-(U2-CONT)")
+	(net 6 "Net-(U1-SW)")
+	(net 7 "Net-(U1-PG)")
+	(net 8 "Net-(U2-OUT)")
+	(net 9 "Net-(U2-DISCH)")
+	(net 10 "Net-(U3-BASE)")
 	(footprint "LOGO"
 		(layer "F.Cu")
@@
 			(size 0.381 0.9652)
 			(layers "F.Cu" "F.Paste" "F.Mask")
-			(net 4 "Net-(U1-FB)")
+			(net 3 "/+5V")
 			(pinfunction "FB")
 			(pintype "input")
@@
 			(size 0.381 0.9652)
 			(layers "F.Cu" "F.Paste" "F.Mask")
-			(net 8 "Net-(U1-PG)")
+			(net 7 "Net-(U1-PG)")
 			(pinfunction "PG")
 			(pintype "output")
@@
 			(size 0.381 0.9652)
 			(layers "F.Cu" "F.Paste" "F.Mask")
-			(net 7 "Net-(U1-SW)")
+			(net 6 "Net-(U1-SW)")
 			(pinfunction "SW_2")
 			(pintype "output")
@@
 			(size 0.381 0.9652)
 			(layers "F.Cu" "F.Paste" "F.Mask")
-			(net 7 "Net-(U1-SW)")
+			(net 6 "Net-(U1-SW)")
 			(pinfunction "SW")
 			(pintype "output")
@@
 			(size 0.4332 0.329999)
 			(layers "F.Cu" "F.Paste" "F.Mask")
-			(net 5 "Net-(U2-THRES)")
+			(net 4 "Net-(U2-THRES)")
 			(pintype "unspecified")
 		)
@@
 			(size 0.762 0.8128)
 			(layers "F.Cu" "F.Paste" "F.Mask")
-			(net 10 "Net-(U2-DISCH)")
+			(net 9 "Net-(U2-DISCH)")
 			(pintype "unspecified")
 		)
@@
 			(size 0.762 0.8128)
 			(layers "F.Cu" "F.Paste" "F.Mask")
-			(net 7 "Net-(U1-SW)")
+			(net 6 "Net-(U1-SW)")
 			(pintype "unspecified")
 		)
@@
 			(size 0.762 0.8128)
 			(layers "F.Cu" "F.Paste" "F.Mask")
-			(net 8 "Net-(U1-PG)")
+			(net 7 "Net-(U1-PG)")
 			(pintype "unspecified")
 		)
@@
 			(size 0.6096 0.508)
 			(layers "F.Cu" "F.Paste" "F.Mask")
-			(net 6 "Net-(U2-CONT)")
+			(net 5 "Net-(U2-CONT)")
 			(pintype "unspecified")
 		)
@@
 			(size 0.6604 0.508)
 			(layers "F.Cu" "F.Paste" "F.Mask")
-			(net 10 "Net-(U2-DISCH)")
+			(net 9 "Net-(U2-DISCH)")
 			(pintype "unspecified")
 		)
@@
 			(size 0.6604 0.508)
 			(layers "F.Cu" "F.Paste" "F.Mask")
-			(net 5 "Net-(U2-THRES)")
+			(net 4 "Net-(U2-THRES)")
 			(pintype "unspecified")
 		)
@@
 			(size 1.9812 0.5588)
 			(layers "F.Cu" "F.Paste" "F.Mask")
-			(net 5 "Net-(U2-THRES)")
+			(net 4 "Net-(U2-THRES)")
 			(pinfunction "TRIG")
 			(pintype "input")
@@
 			(size 1.9812 0.5588)
 			(layers "F.Cu" "F.Paste" "F.Mask")
-			(net 9 "Net-(U2-OUT)")
+			(net 8 "Net-(U2-OUT)")
 			(pinfunction "OUT")
 			(pintype "output")
@@
 			(size 1.9812 0.5588)
 			(layers "F.Cu" "F.Paste" "F.Mask")
-			(net 6 "Net-(U2-CONT)")
+			(net 5 "Net-(U2-CONT)")
 			(pinfunction "CONT")
 			(pintype "unspecified")
@@
 			(size 1.9812 0.5588)
 			(layers "F.Cu" "F.Paste" "F.Mask")
-			(net 5 "Net-(U2-THRES)")
+			(net 4 "Net-(U2-THRES)")
 			(pinfunction "THRES")
 			(pintype "input")
@@
 			(size 1.9812 0.5588)
 			(layers "F.Cu" "F.Paste" "F.Mask")
-			(net 10 "Net-(U2-DISCH)")
+			(net 9 "Net-(U2-DISCH)")
 			(pinfunction "DISCH")
 			(pintype "unspecified")
@@
 			(size 1.397 2.8956)
 			(layers "F.Cu" "F.Paste" "F.Mask")
-			(net 4 "Net-(U1-FB)")
+			(net 1 "GND")
 			(pintype "unspecified")
 		)
@@
 			(size 0.755599 0.799998)
 			(layers "F.Cu" "F.Paste" "F.Mask")
-			(net 9 "Net-(U2-OUT)")
+			(net 8 "Net-(U2-OUT)")
 			(pintype "unspecified")
 		)
@@
 			(size 0.755599 0.799998)
 			(layers "F.Cu" "F.Paste" "F.Mask")
-			(net 11 "Net-(U3-BASE)")
+			(net 10 "Net-(U3-BASE)")
 			(pintype "unspecified")
 		)
@@
 			(size 3.8608 5.5118)
 			(layers "F.Cu" "F.Paste" "F.Mask")
-			(net 7 "Net-(U1-SW)")
+			(net 6 "Net-(U1-SW)")
 			(pinfunction "1")
 			(pintype "unspecified")
@@
 			(size 0.4826 1.6383)
 			(layers "F.Cu" "F.Paste" "F.Mask")
-			(net 11 "Net-(U3-BASE)")
+			(net 10 "Net-(U3-BASE)")
 			(pinfunction "BASE")
 			(pintype "unspecified")
@@
 		(fill solid)
 		(layer "F.Cu")
-		(net 7)
+		(net 6)
 	)
 	(gr_curve
@@
 		(fill solid)
 		(layer "F.Cu")
-		(net 11)
+		(net 10)
 	)
 	(gr_curve
@@
 		(fill solid)
 		(layer "F.Cu")
-		(net 8)
+		(net 7)
 	)
 	(gr_rect
@@
 		(fill solid)
 		(layer "F.Cu")
-		(net 7)
+		(net 6)
 	)
 	(gr_curve
@@
 		(fill solid)
 		(layer "F.Cu")
-		(net 5)
+		(net 4)
 	)
 	(gr_curve
@@
 		(fill solid)
 		(layer "F.Cu")
-		(net 10)
+		(net 9)
 	)
 	(gr_curve
@@
 		(fill solid)
 		(layer "F.Cu")
-		(net 5)
+		(net 4)
 	)
 	(gr_curve
@@
 	)
 	(gr_rect
-		(start 132.7 78.5)
+		(start 132.65 78.5)
 		(end 133.45 81.9)
 		(stroke
@@
 		(fill solid)
 		(layer "F.Cu")
-		(net 6)
+		(net 5)
 	)
 	(gr_curve
@@
 		(net 3)
 	)
+	(gr_rect
+		(start 132.35 80.14)
+		(end 132.81 80.69)
+		(stroke
+			(width 0.2)
+			(type solid)
+		)
+		(fill solid)
+		(layer "F.Cu")
+		(net 2)
+	)
 	(gr_curve
 		(pts
@@
 		(fill solid)
 		(layer "F.Cu")
-		(net 5)
+		(net 4)
 	)
 	(gr_curve
@@
 		(fill solid)
 		(layer "F.Cu")
-		(net 5)
+		(net 4)
 	)
 	(gr_curve
@@
 		(net 3)
 	)
-	(gr_poly
-		(pts
-			(xy 133.3 77.15) (xy 135.5 77.15) (xy 135.5 77.4) (xy 133.3 77.4)
-		)
-		(stroke
-			(width 0.2)
-			(type solid)
-		)
-		(fill solid)
-		(layer "F.Cu")
-		(net 4)
-	)
 	(gr_curve
 		(pts
@@
 		(fill solid)
 		(layer "F.Cu")
-		(net 5)
+		(net 4)
 	)
 	(gr_curve
@@
 		(net 3)
 	)
+	(gr_rect
+		(start 133.58 75.91)
+		(end 136.14 76.72)
+		(stroke
+			(width 0.2)
+			(type solid)
+		)
+		(fill solid)
+		(layer "F.Cu")
+		(net 1)
+	)
 	(gr_curve
 		(pts
@@
 		(fill solid)
 		(layer "F.Cu")
-		(net 5)
+		(net 4)
 	)
 	(gr_poly
@@
 		(fill solid)
 		(layer "F.Cu")
-		(net 11)
+		(net 10)
 	)
 	(gr_curve
@@
 		(net 3)
 	)
+	(gr_poly
+		(pts
+			(xy 133.28 77.15) (xy 134.98 77.15) (xy 134.98 78.72) (xy 139.07 78.72) (xy 139.1 79.32) (xy 134.66 79.3)
+			(xy 134.66 77.39) (xy 133.29 77.39) (xy 133.27 77.16)
+		)
+		(stroke
+			(width 0.2)
+			(type solid)
+		)
+		(fill solid)
+		(layer "F.Cu")
+		(net 3)
+	)
 	(gr_curve
 		(pts
@@
 		(width 0.2)
 		(layer "F.Cu")
-		(net 9)
+		(net 8)
 	)
 	(segment
@@
 		(width 0.2)
 		(layer "F.Cu")
-		(net 9)
+		(net 8)
 	)
 	(segment
@@
 		(width 0.2)
 		(layer "F.Cu")
-		(net 9)
+		(net 8)
 	)
 	(group ""
